File: Work.kicad_sch (KiCad schematic)
At the start: 1 part, among them J3 ZX62R-B-5P_30_

Commit message: SCH & PCB Data
Parts:
- removed J3: ZX62R-B-5P_30_, HLDC_E1:ZX62R-B-5P_30, symbol HLDC_E1:ZX62R-B-5P_30_
- added TP5: TP_FL, HLDC_E1:HLDC_logo2, symbol HLDC_E1:TP_FL
Connections:
- no-connect marks 0 -> 1
Other:
- added sheet IR (IR.kicad_sch)
- added sheet Main (Main.kicad_sch)
- added sheet Power (Power.kicad_sch)
- added sheet Radar (Radar.kicad_sch)
- added sheet Serial (Serial.kicad_sch)
